Commit message: updated

File: avp_teleoperate/assets/g1/g1_body29_inspired_hand.urdf (robot description, URDF)
Before this commit: robot g1, 65 links, 64 joints
Links:
- removed link L_index_tip_cube
- removed link R_index_tip_cube
Joints:
- joint L_index_tip_joint: child L_index_tip_cube -> (none)
- joint R_index_tip_joint: child R_index_tip_cube -> (none)

Commit message: updated

File: avp_teleoperate/assets/g1/g1_body29_inspired_hand.urdf (robot description, URDF)
Before this commit: robot g1, 63 links, 64 joints
Links:
- added link L_index_tip; visual sphere radius=0.005
- added link R_index_tip; visual sphere radius=0.005
Joints:
- joint L_index_tip_joint: child (none) -> L_index_tip
- joint R_index_tip_joint: child (none) -> R_index_tip
